Commit message: Simple lateral jump kinda works

File: solo_12/urdf/solo_12.urdf (robot description, URDF)
Before this commit: robot solo_12, 16 links, 15 joints
Links:
- added link worldRX
- added link worldRY
- added link worldY
Joints:
- added joint CHEAT_MODE_RX: type revolute, parent worldRX, child worldX, origin xyz=0 0 0 rpy=0 0 0, axis 1 0 0, limit lower=0 upper=0 effort=0 velocity=0
- added joint CHEAT_MODE_RY: type revolute, parent worldRY, child worldRX, origin xyz=0 0 0 rpy=0 0 0, axis 0 1 0, limit lower=0 upper=0 effort=0 velocity=0
- added joint CHEAT_MODE_Y: type prismatic, parent worldY, child worldZ, origin xyz=0 0 0 rpy=0 0 0, axis 0 1 0, limit lower=0 upper=0 effort=0 velocity=0
- joint CHEAT_MODE_RZ: child worldX -> worldRY
- joint CHEAT_MODE_X: child worldZ -> worldY

Commit message: uhhhhhhhhh

File: solo_12/urdf/solo_12.urdf (robot description, URDF)
Before this commit: robot solo_12, 19 links, 18 joints
Joints:
- joint CHEAT_MODE_RX: child worldX -> worldRY
- joint CHEAT_MODE_RY: child worldRX -> base_link
- joint CHEAT_MODE_RZ: child worldRY -> worldRX
- joint CHEAT_MODE_Z: child base_link -> worldRZ
