Commit message: savingchanges

File: huron/huron_description/urdf/huron.urdf (robot description, URDF)
Before this commit: robot huron, 16 links, 15 joints
Links:
- removed link base_link
- added link L_FOOT, mass 0.01; visual box size=0.078 0.005 0.221
- added link R_FOOT, mass 0.01; visual box size=0.078 0.005 0.221
- added link body
- added link dummy, mass 0.000863223621815312
- added link l1_foot_ft_link, mass 0.0086322; visual mesh filename=package://huron_description/meshes/stl_meshes/l_foot_ft.STL scale=1 1 1
- added link l2_foot_ft_link, mass 0.00863223621815312; visual mesh filename=package://huron_description/meshes/stl_meshes/l_foot_ft.STL scale=1 1 1
- added link l3_foot_ft_link, mass 0.00863223621815312; visual mesh filename=package://huron_description/meshes/stl_meshes/l_foot_ft.STL scale=1 1 1
- added link l4_foot_ft_link, mass 0.00863223621815312; visual mesh filename=package://huron_description/meshes/stl_meshes/l_foot_ft.STL scale=1 1 1
- added link l_foot_v_ft_link
- added link r1_foot_ft_link, mass 0.0086322; visual mesh filename=package://huron_description/meshes/stl_meshes/r_foot_ft.STL scale=1 1 1
- added link r2_foot_ft_link, mass 0.00863223621815318; visual mesh filename=package://huron_description/meshes/stl_meshes/r_foot_ft.STL scale=1 1 1
- added link r3_foot_ft_link, mass 0.00863223621815318; visual mesh filename=package://huron_description/meshes/stl_meshes/r_foot_ft.STL scale=1 1 1
- added link r4_foot_ft_link, mass 0.00863223621815318; visual mesh filename=package://huron_description/meshes/stl_meshes/r_foot_ft.STL scale=1 1 1
- added link r_foot_v_ft_link
- link base_footprint: geometry visual mesh filename=package://huron_description/meshes/stl_meshes/base_link.STL scale=1 1 1
- link battery_link: geometry visual box size=0.065 0.188 0.151
- link l_ankle_pitch_link: geometry visual mesh filename=package://huron_description/meshes/stl_meshes/l_ankle_pitch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 scale=1 1 1
- link l_ankle_roll_link: mass 1.8633 -> 1.8533; geometry visual mesh filename=package://huron_description/meshes/stl_meshes/l_ankle_roll_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 scale=1 1 1
- link l_hip_pitch_link: geometry visual mesh filename=package://huron_description/meshes/stl_meshes/l_hip_pitch_l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 scale=1 1 1
- link l_hip_roll_link: geometry visual mesh filename=package://huron_description/meshes/stl_meshes/l_hip_roll_li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 scale=1 1 1
- link l_hip_yaw_link: geometry visual mesh filename=package://huron_description/meshes/stl_meshes/l_hip_yaw_lin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 scale=1 1 1
- link l_knee_pitch_link: geometry visual mesh filename=package://huron_description/meshes/stl_meshes/l_knee_pitch_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 scale=1 1 1
- link r_ankle_pitch_link: geometry visual mesh filename=package://huron_description/meshes/stl_meshes/r_ankle_pitch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 scale=1 1 1
- link r_ankle_roll_link: mass 1.8633 -> 1.8533; geometry visual mesh filename=package://huron_description/meshes/stl_meshes/r_ankle_roll_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 scale=1 1 1
- link r_hip_pitch_link: geometry visual mesh filename=package://huron_description/meshes/stl_meshes/r_hip_pitch_l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 scale=1 1 1
- link r_hip_roll_link: geometry visual mesh filename=package://huron_description/meshes/stl_meshes/r_hip_roll_li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 scale=1 1 1
- link r_hip_yaw_link: geometry visual mesh filename=package://huron_description/meshes/stl_meshes/r_hip_yaw_lin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 scale=1 1 1
- link r_knee_pitch_link: geometry visual mesh filename=package://huron_description/meshes/stl_meshes/r_knee_pitch_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 scale=1 1 1
Joints:
- added joint dummy_fixed: type fixed, parent dummy, child base_footprint, origin xyz=0 0 0 rpy=0 0 0
- added joint l1_ft_fixed: type fixed, parent l_ankle_roll_link, child l1_foot_ft_link, origin xyz=0.098328 0.020682 0.12788 rpy=-0.024938 0.00629 1.5706, axis 0 0 1
- added joint l2_ft_fixed: type fixed, parent l_ankle_roll_link, child l2_foot_ft_link, origin xyz=0.098275 -0.014318 0.12788 rpy=-0.024938 0.00629 1.5706, axis 0 0 1
- added joint l3_ft_fixed: type fixed, parent l_ankle_roll_link, child l3_foot_ft_link, origin xyz=0.098272 -0.016649 0 rpy=-0.024938 0.00629 1.5706, axis 0 0 1
- added joint l4_ft_fixed: type fixed, parent l_ankle_roll_link, child l4_foot_ft_link, origin xyz=0.098322 0.01686 0 rpy=-0.024938 0.00629 1.5706, axis 0 0 1
- added joint l_foot_base_fixed: type fixed, parent l1_foot_ft_link, child L_FOOT, origin xyz=-0.0175 -0.0025 -0.06395 rpy=0 0 0
- added joint lv_ft_fixed: type fixed, parent l4_foot_ft_link, child l_foot_v_ft_link, origin xyz=0.045 0.0 0.0 rpy=0 -1.570796327 0
- added joint r1_ft_fixed: type fixed, parent r_ankle_roll_link, child r1_foot_ft_link, origin xyz=0.098271 0.014348 0.12788 rpy=-0.0095317 0.011124 1.5707, axis 0 0 1
- added joint r2_ft_fixed: type fixed, parent r_ankle_roll_link, child r2_foot_ft_link, origin xyz=0.098334 -0.020652 0.12788 rpy=-0.0095317 0.011124 1.5707, axis 0 0 1
- added joint r3_ft_fixed: type fixed, parent r_ankle_roll_link, child r3_foot_ft_link, origin xyz=0.098328 -0.01683 0 rpy=-0.0095317 0.011124 1.5707, axis 0 0 1
- added joint r4_ft_fixed: type fixed, parent r_ankle_roll_link, child r4_foot_ft_link, origin xyz=0.098267 0.016679 0 rpy=-0.0095317 0.011124 1.5707, axis 0 0 1
- added joint r_foot_base_fixed: type fixed, parent r1_foot_ft_link, child R_FOOT, origin xyz=-0.0175 -0.0025 -0.06395 rpy=0 0 0
- added joint rv_ft_fixed: type fixed, parent r4_foot_ft_link, child r_foot_v_ft_link, origin xyz=0.0 0.0 0.0 rpy=0 0 0, axis 0 0 0
- joint base_fixed: child base_footprint -> dummy; origin xyz=0 0 0 rpy=0 0 0 -> xyz=0 0 1.1318 rpy=0 0 0; parent base_link -> body
- joint l_ankle_pitch_joint: limit lower=-0.5236 upper=0.1745 effort=1000 velocity=3 -> lower=-3.1416 upper=3.1416 effort=1000 velocity=40; origin xyz=0.37 0 0 rpy=0 0 0.0 -> xyz=0.3715 3.1633E-05 0.0025 rpy=0 0 0.0; type revolute -> continuous
- joint l_ankle_roll_joint: limit lower=-0.3491 upper=0.3491 effort=1000 velocity=3 -> lower=-3.1416 upper=3.1416 effort=1000 velocity=40; type revolute -> continuous
- joint l_hip_pitch_joint: limit lower=-1.2217 upper=1.2217 effort=1000 velocity=3 -> lower=-3.1416 upper=3.1416 effort=1000 velocity=40; origin xyz=1.6665E-05 -0.0165 -5E-05 rpy=-1.570796327 0 -1.570796327 -> xyz=0 0 0 rpy=-1.570796327 0 -1.570796327; type revolute -> continuous
- joint l_hip_roll_joint: limit lower=-0.01 upper=0.5236 effort=1000 velocity=3 -> lower=-3.1416 upper=3.1416 effort=1000 velocity=40; type revolute -> continuous
- joint l_hip_yaw_joint: limit lower=-3.1416 upper=3.1416 effort=1000 velocity=3 -> lower=-3.1416 upper=3.1416 effort=1000 velocity=40; origin xyz=-0.0775000000000011 0 -0.1451242 rpy=0 0 0 -> xyz=-0.0775 0 -0.14512 rpy=0 0 -0.0; type revolute -> continuous
- joint l_knee_pitch_joint: limit lower=-1.570796327 upper=1.570796327 effort=1000 velocity=3 -> lower=-3.1416 upper=3.1416 effort=1000 velocity=40; origin xyz=0.49628 0 0 rpy=0 0 0 -> xyz=0.512778478308813 5.00027201116859E-05 1.66647320003488E-05 rpy=0 0 0; type revolute -> continuous
- joint r_ankle_pitch_joint: limit lower=-0.5236 upper=0.1745 effort=1000 velocity=3 -> lower=-3.1416 upper=3.1416 effort=1000 velocity=40; origin xyz=0.37 0 0 rpy=0 0 0.0 -> xyz=0.370000000000006 -3.16358749707368E-05 -0.00249999999999943 rpy=0 0 0.0; type revolute -> continuous
- joint r_ankle_roll_joint: limit lower=-0.3491 upper=0.3491 effort=1000 velocity=3 -> lower=-3.1416 upper=3.1416 effort=1000 velocity=40; type revolute -> continuous
- joint r_hip_pitch_joint: limit lower=-1.2217 upper=1.2217 effort=1000 velocity=3 -> lower=-3.1416 upper=3.1416 effort=1000 velocity=40; origin xyz=-1.6665E-05 -0.0165 -5E-05 rpy=-1.570796327 0 -1.570796327 -> xyz=0 0 0 rpy=-1.570796327 0 -1.570796327; type revolute -> continuous
- joint r_hip_roll_joint: limit lower=-0.5236 upper=0.01 effort=1000 velocity=3 -> lower=-3.1416 upper=3.1416 effort=1000 velocity=40; type revolute -> continuous
- joint r_hip_yaw_joint: limit lower=-3.1416 upper=3.1416 effort=1000 velocity=3 -> lower=-3.1416 upper=3.1416 effort=1000 velocity=40; origin xyz=0.0775 0 -0.14512 rpy=0 0 3.141592654 -> xyz=0.0774999999999944 0 -0.1451242 rpy=0 0 3.141592654; type revolute -> continuous
- joint r_knee_pitch_joint: limit lower=-1.570796327 upper=1.570796327 effort=1000 velocity=3 -> lower=-3.1416 upper=3.1416 effort=1000 velocity=40; origin xyz=0.49628 0 0 rpy=0 0 0 -> xyz=0.512778478308813 4.99999999867273E-05 -1.66647320091612E-05 rpy=0 0 0; type revolute -> continuous
