Commit message: saving progress

File: huron/huron.urdf (robot description, URDF)
Before this commit: robot huron, 16 links, 15 joints
Joints:
- joint l_ankle_pitch_joint: limit lower=-0.5236 upper=0.1745 effort=1000000 velocity=3000 -> lower=-3.1416 upper=3.1416 effort=1000000 velocity=3000
- joint l_ankle_roll_joint: limit lower=-0.3491 upper=0.3491 effort=1000000 velocity=3000 -> lower=-3.1416 upper=3.1416 effort=1000000 velocity=3000
- joint l_hip_pitch_joint: limit lower=-1.2217 upper=1.2217 effort=1000000 velocity=3000 -> lower=-3.1416 upper=3.1416 effort=1000000 velocity=3000
- joint l_hip_roll_joint: limit lower=-0.01 upper=0.5236 effort=1000000 velocity=3000 -> lower=-3.1416 upper=3.1416 effort=1000000 velocity=3000
- joint l_knee_pitch_joint: limit lower=-1.570796327 upper=1.570796327 effort=1000000 velocity=3000 -> lower=-3.1416 upper=3.1416 effort=1000000 velocity=3000
- joint r_ankle_pitch_joint: limit lower=-0.5236 upper=0.1745 effort=1000000 velocity=3000 -> lower=-3.1416 upper=3.1416 effort=1000000 velocity=3000
- joint r_ankle_roll_joint: limit lower=-0.3491 upper=0.3491 effort=1000000 velocity=3000 -> lower=-3.1416 upper=3.1416 effort=1000000 velocity=3000
- joint r_hip_pitch_joint: limit lower=-1.2217 upper=1.2217 effort=1000000 velocity=3000 -> lower=-3.1416 upper=3.1416 effort=1000000 velocity=3000
- joint r_hip_roll_joint: limit lower=-0.5236 upper=0.01 effort=1000000 velocity=3000 -> lower=-3.1416 upper=3.1416 effort=1000000 velocity=3000
- joint r_knee_pitch_joint: limit lower=-1.570796327 upper=1.570796327 effort=1000000 velocity=3000 -> lower=-3.1416 upper=3.1416 effort=1000000 velocity=3000

File: huron/huron_cheat.urdf (robot description, URDF)
Before this commit: robot huron, 22 links, 21 joints
Joints:
- joint l_ankle_pitch_joint: limit lower=-0.5236 upper=0.1745 effort=1000000 velocity=3000 -> lower=-3.1416 upper=3.1416 effort=1000000 velocity=3000
- joint l_ankle_roll_joint: limit lower=-0.3491 upper=0.3491 effort=1000000 velocity=3000 -> lower=-3.1416 upper=3.1416 effort=1000000 velocity=3000
- joint l_hip_pitch_joint: limit lower=-1.2217 upper=1.2217 effort=1000000 velocity=3000 -> lower=-3.1416 upper=3.1416 effort=1000000 velocity=3000
- joint l_hip_roll_joint: limit lower=-0.01 upper=0.5236 effort=1000000 velocity=3000 -> lower=-3.1416 upper=3.1416 effort=1000000 velocity=3000
- joint l_knee_pitch_joint: limit lower=-1.570796327 upper=1.570796327 effort=1000000 velocity=3000 -> lower=-3.1416 upper=3.1416 effort=1000000 velocity=3000
- joint r_ankle_pitch_joint: limit lower=-0.5236 upper=0.1745 effort=1000000 velocity=3000 -> lower=-3.1416 upper=3.1416 effort=1000000 velocity=3000
- joint r_ankle_roll_joint: limit lower=-0.3491 upper=0.3491 effort=1000000 velocity=3000 -> lower=-3.1416 upper=3.1416 effort=1000000 velocity=3000
- joint r_hip_pitch_joint: limit lower=-1.2217 upper=1.2217 effort=1000000 velocity=3000 -> lower=-3.1416 upper=3.1416 effort=1000000 velocity=3000
- joint r_hip_roll_joint: limit lower=-0.5236 upper=0.01 effort=1000000 velocity=3000 -> lower=-3.1416 upper=3.1416 effort=1000000 velocity=3000
- joint r_knee_pitch_joint: limit lower=-1.570796327 upper=1.570796327 effort=1000000 velocity=3000 -> lower=-3.1416 upper=3.1416 effort=1000000 velocity=3000

File: solo_12/urdf/solo_12_leg.urdf (robot description, URDF)
Before this commit: robot solo_12_leg, 4 links, 3 joints
Links:
- added link worldRX
- added link worldRY
- added link worldRZ
- added link worldX
- added link worldY
- added link worldZ
Joints:
- added joint CHEAT_MODE_RX: type revolute, parent worldRX, child worldRY, origin xyz=0 0 0 rpy=0 0 0, axis 1 0 0, limit lower=0 upper=0 effort=0 velocity=0
- added joint CHEAT_MODE_RY: type revolute, parent worldRY, child base_link, origin xyz=0 0 0 rpy=0 0 0, axis 0 1 0, limit lower=0 upper=0 effort=0 velocity=0
- added joint CHEAT_MODE_RZ: type revolute, parent worldRZ, child worldRX, origin xyz=0 0 0 rpy=0 0 0, axis 0 0 1, limit lower=0 upper=0 effort=0 velocity=0
- added joint CHEAT_MODE_X: type prismatic, parent worldX, child worldY, origin xyz=0 0 0 rpy=0 0 0, axis 1 0 0, limit lower=0 upper=0 effort=0 velocity=0
- added joint CHEAT_MODE_Y: type prismatic, parent worldY, child worldZ, origin xyz=0 0 0 rpy=0 0 0, axis 0 1 0, limit lower=0 upper=0 effort=0 velocity=0
- added joint CHEAT_MODE_Z: type prismatic, parent worldZ, child worldRZ, origin xyz=0 0 0 rpy=0 0 0, axis 0 0 1, limit lower=0 upper=0 effort=0 velocity=0

Commit message: Revert "saving progress"
This reverts commit 55a1a5de3c290b3da9a60e76fff4f91f0c205a23.

File: huron/huron.urdf (robot description, URDF)
Before this commit: robot huron, 16 links, 15 joints
Joints:
- joint l_ankle_pitch_joint: limit lower=-3.1416 upper=3.1416 effort=1000000 velocity=3000 -> lower=-0.5236 upper=0.1745 effort=1000000 velocity=3000
- joint l_ankle_roll_joint: limit lower=-3.1416 upper=3.1416 effort=1000000 velocity=3000 -> lower=-0.3491 upper=0.3491 effort=1000000 velocity=3000
- joint l_hip_pitch_joint: limit lower=-3.1416 upper=3.1416 effort=1000000 velocity=3000 -> lower=-1.2217 upper=1.2217 effort=1000000 velocity=3000
- joint l_hip_roll_joint: limit lower=-3.1416 upper=3.1416 effort=1000000 velocity=3000 -> lower=-0.01 upper=0.5236 effort=1000000 velocity=3000
- joint l_knee_pitch_joint: limit lower=-3.1416 upper=3.1416 effort=1000000 velocity=3000 -> lower=-1.570796327 upper=1.570796327 effort=1000000 velocity=3000
- joint r_ankle_pitch_joint: limit lower=-3.1416 upper=3.1416 effort=1000000 velocity=3000 -> lower=-0.5236 upper=0.1745 effort=1000000 velocity=3000
- joint r_ankle_roll_joint: limit lower=-3.1416 upper=3.1416 effort=1000000 velocity=3000 -> lower=-0.3491 upper=0.3491 effort=1000000 velocity=3000
- joint r_hip_pitch_joint: limit lower=-3.1416 upper=3.1416 effort=1000000 velocity=3000 -> lower=-1.2217 upper=1.2217 effort=1000000 velocity=3000
- joint r_hip_roll_joint: limit lower=-3.1416 upper=3.1416 effort=1000000 velocity=3000 -> lower=-0.5236 upper=0.01 effort=1000000 velocity=3000
- joint r_knee_pitch_joint: limit lower=-3.1416 upper=3.1416 effort=1000000 velocity=3000 -> lower=-1.570796327 upper=1.570796327 effort=1000000 velocity=3000

File: huron/huron_cheat.urdf (robot description, URDF)
Before this commit: robot huron, 22 links, 21 joints
Joints:
- joint l_ankle_pitch_joint: limit lower=-3.1416 upper=3.1416 effort=1000000 velocity=3000 -> lower=-0.5236 upper=0.1745 effort=1000000 velocity=3000
- joint l_ankle_roll_joint: limit lower=-3.1416 upper=3.1416 effort=1000000 velocity=3000 -> lower=-0.3491 upper=0.3491 effort=1000000 velocity=3000
- joint l_hip_pitch_joint: limit lower=-3.1416 upper=3.1416 effort=1000000 velocity=3000 -> lower=-1.2217 upper=1.2217 effort=1000000 velocity=3000
- joint l_hip_roll_joint: limit lower=-3.1416 upper=3.1416 effort=1000000 velocity=3000 -> lower=-0.01 upper=0.5236 effort=1000000 velocity=3000
- joint l_knee_pitch_joint: limit lower=-3.1416 upper=3.1416 effort=1000000 velocity=3000 -> lower=-1.570796327 upper=1.570796327 effort=1000000 velocity=3000
- joint r_ankle_pitch_joint: limit lower=-3.1416 upper=3.1416 effort=1000000 velocity=3000 -> lower=-0.5236 upper=0.1745 effort=1000000 velocity=3000
- joint r_ankle_roll_joint: limit lower=-3.1416 upper=3.1416 effort=1000000 velocity=3000 -> lower=-0.3491 upper=0.3491 effort=1000000 velocity=3000
- joint r_hip_pitch_joint: limit lower=-3.1416 upper=3.1416 effort=1000000 velocity=3000 -> lower=-1.2217 upper=1.2217 effort=1000000 velocity=3000
- joint r_hip_roll_joint: limit lower=-3.1416 upper=3.1416 effort=1000000 velocity=3000 -> lower=-0.5236 upper=0.01 effort=1000000 velocity=3000
- joint r_knee_pitch_joint: limit lower=-3.1416 upper=3.1416 effort=1000000 velocity=3000 -> lower=-1.570796327 upper=1.570796327 effort=1000000 velocity=3000

File: solo_12/urdf/solo_12_leg.urdf (robot description, URDF)
Before this commit: robot solo_12_leg, 10 links, 9 joints
Links:
- removed link worldRX
- removed link worldRY
- removed link worldRZ
- removed link worldX
- removed link worldY
- removed link worldZ
Joints:
- removed joint CHEAT_MODE_RX
- removed joint CHEAT_MODE_RY
- removed joint CHEAT_MODE_RZ
- removed joint CHEAT_MODE_X
- removed joint CHEAT_MODE_Y
- removed joint CHEAT_MODE_Z
